Commit message: Remove unnecessary flange frame

File: robot_specific_config/abb_irb4600_support/urdf/irb4600_60_205_macro.xacro (robot description, xacro)
@@ -154,16 +154,9 @@
       <child link="${prefix}base"/>
     </joint>
-    <!-- ROS-Industrial 'flange' frame- attachment point for EEF models -->
-    <link name="${prefix}flange"/>
-    <joint type="fixed" name="${prefix}joint_6-flange">
-      <origin xyz="0 0 0" rpy="0 0 0"/>
-      <parent link="${prefix}link_6"/>
-      <child link="${prefix}flange"/>
-    </joint>
     <!-- ROS-Industrial 'tool0' frame- all-zeros tool frame -->
     <link name="${prefix}tool0" />
     <joint name="${prefix}link_6-tool0" type="fixed">
       <origin xyz="0 0 0" rpy="0 ${radians(90)} 0" />
-      <parent link="${prefix}flange" />
+      <parent link="${prefix}link_6" />
       <child link="${prefix}tool0" />
     </joint>
